File: _restore_backup_2026-06-18T18-26-54-256/eis_pcb.kicad_sch (KiCad schematic)
At the start: 69 parts, among them J1 527451897, J12 104031-0811, J2 GSB1C41110SSHR, J4 541020164, P1 V.BATT, P2 GND.BATT, Q3 IRLML6344TRPBF, SW1 SWT0210-045026GSA, SW2 SWT0210-045026GSA_REVA, U1 ESP32-S3-WROOM-1-N8R8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

Commit message: remove 2.8v circuitry
turns out it wasnt need it. my chud life
Parts:
- removed J1: 527451897, CON_527451897_MOL, symbol 2026-06-19_01-22-01:527451897
- added J13: 10051922-1810ELF, 10051922-1810ELF:AMPHENOL_10051922-1810ELF, symbol 10051922-1810ELF:10051922-1810ELF
- added U8: TPS7A0328PYCHR, YCH0004-IPC_A, symbol 2026-06-18_22-09-09:TPS7A0328PYCHR
- C12, C26: value 0.1u -> 100n
- renumbered U2 to U1, U4 to U2, U1 to U3, U6 to U5, U3 to U6, U5 to U7
Connections:
- net +3V3: now also R16.1, J13.17, J13.4
- net +VSYS: now also U8.1 (IN)
- net CS.SCREEN: now also J13.8
- net CTP_INT: now also J13.16
- net CTP_RST: now also J13.15
- net CTP_SCL: now also J13.13
- net CTP_SDA: now also J13.14
- net DC: now also J13.7
- net GND: now also J13.1, J13.12, J13.18, J13.5, J13.6, U8.4 (GND); no longer R20.2
- net K: now also Q3.3, J13.2; no longer R16.2
- net MOSI: now also J13.10
- net PWR.EN: now also U8.3 (EN)
- net SCLK: now also J13.9
- net SCREEN.RST: now also J13.11
- net at R20.1: no longer U7.15 (SYSOFF)
- new net: J13.3, R16.2
- new net +2V8: U8.2 (OUT)
- new net SYSOFF: U7.15 (SYSOFF)
Other:
- note added: "2.8V LDO"
- moved on the sheet: Q3, R14, R16, R2, R20
